File: pcb/ser2can.brd (EAGLE design)
At the start: 80.7 x 40.7 mm, 67 parts, among them Q1 8MHz, Q2 32768Hz, SW1 KSS-2EG4430, X1 MSTBA4

Commit message: sch&pcb some modifications
Parts:
- removed SW1: KSS-2EG4430, buttons:KSS-2EG4430
- removed X3: (no value), pinhead-fixdrills:1X05M
- added JP3: (no value), pinhead-fixdrills:1X02SMALL
- added SWD: SWD-6, jtag:JTAG6PIN
- JP2: device pinhead-fixdrills:1X02M -> pinhead-fixdrills:1X02SMALL
- moved R6 8.98 mm to (64.1, 6.35)
- moved TP4 4.51 mm to (20.6, 25.4)
- moved R7 3.18 mm to (54.0, 12.7)
- moved C14 1.93 mm to (29.5, 32.7), turned to 90 degrees
- moved R18 1.93 mm to (41.3, 8.89)
- moved C10 1.80 mm to (19.1, 25.4)
- moved C8 1.27 mm to (64.1, 30.5)
- moved JP2 1.27 mm to (42.5, 6.35)
- moved R15 0.90 mm to (11.4, 11.4)
- moved C17 0.90 mm to (17.1, 10.2)
- moved R19 0.64 mm to (44.5, 8.89)
- moved C20 0.63 mm to (32.4, 11.1)
- moved LED4 0.63 mm to (2.54, 11.4)
Connections:
- new net PA15: DD2.38, X2.20
- net !RESET: now also SWD.5; no longer SW1.2, X3.4
- net +3V3: now also SWD.1; no longer X3.1
- net CAN_L: now also JP3.1
- net CAN_L_R: now also JP3.2
- net GND: now also SWD.3; no longer SW1.1, X2.20, X3.5
- net SWCLK: now also SWD.2; no longer X3.3
- net SWDIO: now also SWD.4; no longer X3.2
Routing:
- net PA15: track 0.00 -> 26.5 mm, vias 0 -> 2
- net CAN_L: track 5.19 -> 29.0 mm
- net CAN_L_R: track 8.49 -> 26.4 mm
- net ISOVCC: track 55.2 -> 42.5 mm
- net N$6: track 2.63 -> 11.7 mm
- net !RESET: track 50.9 -> 46.1 mm, vias 3 -> 4
- net +3V3: track 125.3 -> 121.0 mm, vias 5 -> 4
- net N$3: track 5.46 -> 9.64 mm
- net SWDIO: track 23.8 -> 26.4 mm, vias 0 -> 1
- net N$2: track 6.32 -> 4.20 mm
- net !CPRST: track 20.1 -> 21.8 mm
- net PB3: track 26.1 -> 27.7 mm, vias 1 -> 2
- net !SUSPEND: track 16.7 -> 18.2 mm
- net +5V: track 92.2 -> 93.5 mm
- net BOOT1: track 25.3 -> 26.6 mm, vias 0 -> 2
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Other:
- board text added: "PA15"
- board text added: "Rev.B (07/14)"
- board text removed: "Rev.B (04/13)"
- board text removed: "SWD"

Commit message: little changes. pictures
Parts:
- removed JP3: (no value), pinhead-fixdrills:1X02SMALL
- added C23: 100uF/6.3V, rc-master-smd:SMC_C
- added R21: 330, rc-master-smd:R0603
- added SW1: KSS-2EG4430, buttons:KSS-2EG4430
- C1: value 560pF -> 10uF
- C10: value 0.1 -> 22pF
- C11, C12: value 22pF -> 0.1
- C15: value 0.1 -> (none); device rc-master-smd:C0603 -> rc-master:C050-110X055
- C17: value 0.1 -> 100uF/6.3V; device rc-master-smd:C0805 -> rc-master-smd:SMC_C
- C18: device rc-master-smd:C0805 -> rc-master-smd:C0603
- C19: value 100uF/6.3V -> 560pF; device rc-master-smd:SMC_C -> rc-master-smd:C0603
- C2: value 560pF -> 10pF
- C20: value 0.1 -> 560pF
- C21, C22: value 10pF -> 0.1; device rc-master-smd:C0603 -> rc-master-smd:C0805
- C3: value 10uF -> 0.1
- C5: value 0.1 -> 10pF
- C6: value 0.1 -> NC (0.1)
- C7: value 0.1 -> 0.1 (NC)
- C8: value 100uF/6.3V -> 22pF; device rc-master-smd:SMC_C -> rc-master-smd:C0603
- C9: value (none) -> 0.1; device rc-master:C050-110X055 -> rc-master-smd:C0603
- JP2: device pinhead-fixdrills:1X02SMALL -> pinhead-fixdrills:1X02M
- Q1: value 8MHz -> 32768Hz; device discrete:HC49/S -> discrete:MM20SS
- Q2: value 32768Hz -> 8MHz; device discrete:MM20SS -> discrete:HC49/S
- R1: value NC -> 1K
- R10: value 1M -> 330
- R11: value 10 -> 330
- R12: value 330 -> 10K
- R13: value 330 -> NC
- R14: value 10K -> 330
- R15: value 330 -> 0
- R16, R17: value 4.7K -> 100
- R18: value 10K -> 4.7K
- R19: value 1K -> 4.7K
- R2, R3: value 100 -> 10K
- R20: value 1M -> 120; device rc-master-smd:R0603 -> rc-master-smd:R0805
- R4: value 120 -> 1M; device rc-master-smd:R0805 -> rc-master-smd:R0603
- R5: value 0 -> 1M
- R6: value 330 -> 0/FB
- R7: value nc -> 10K; device rc-master-smd:R1206 -> rc-master-smd:R0603
- R8: value 1M -> nc
- R9: value 10K -> 1M; device rc-master-smd:R0603 -> rc-master-smd:R1206
- X1: value MSTBA4 -> (none); device con-phoenix-508:MSTBA4 -> pinhead-fixdrills:2X10
- X2: value (none) -> MSTBA4; device pinhead-fixdrills:2X10 -> con-phoenix-508:MSTBA4
- moved LED1 78.9 mm to (2.54, 32.4), turned to 90 degrees
- moved LED3 77.8 mm to (77.5, 7.62), turned to 270 degrees
- moved R14 55.8 mm to (64.1, 6.35), turned to 0 degrees
- moved C1 52.3 mm to (16.2, 16.2), turned to 270 degrees
- moved R15 51.3 mm to (61.3, 23.5), turned to 270 degrees
- moved C17 51.2 mm to (64.1, 30.5), turned to 0 degrees
- moved R13 48.7 mm to (61.3, 26.7), turned to 90 degrees
- moved X1 47.1 mm to (33.7, 37.5), turned to 180 degrees
- moved X2 47.1 mm to (77.5, 20.3), turned to 90 degrees
- moved C19 44.2 mm to (67.3, 27.3)
- moved C7 42.2 mm to (17.5, 25.4), turned to 270 degrees
- moved C20 34.9 mm to (67.3, 12.1), turned to 0 degrees
- moved R6 33.9 mm to (43.2, 33.0), turned to 180 degrees
- moved R16 33.3 mm to (64.1, 27.3)
- moved R9 32.9 mm to (54.0, 33.0), turned to 0 degrees
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Connections:
- removed net N$11: DD2.2
- new net PC13: DD2.2, R3.2
- net !LCD_CS: now also X1.13; no longer X2.13
- net !RESET: now also C6.2, C7.1, R7.1; no longer C10.2, R9.1
- net +3V3: now also C11.1, C13.1, C22.1, C23.+, C9.1, R18.2, R19.2, R21.2, R6.1, R7.2, SW1.1, X1.1; no longer C14.1, C15.1, C16.1, C19.+, C20.1, JP2.1, R11.1, R15.2, R16.2, R17.2, R9.2, X2.1
- net +5V: now also C1.1, C14.1, C21.1, R8.1; no longer C17.1, C4.1, C6.1, R7.1
- net BOOT0: now also R2.2; no longer R18.2
- net BOOT1: now also R11.1, R12.1; no longer R13.1, R14.1
- net CANH: now also R16.2; no longer R2.2
- net CANL: now also R17.2; no longer R3.2
- net CAN_H: now also R20.1, X2.3; no longer R4.1, X1.3
- net CAN_L: now also JP1.1, X2.2; no longer JP3.1, X1.2
- net CAN_L_R: now also JP1.2, R20.2, X2.1; no longer JP3.2, R4.2, X1.1
- net DTR: now also C6.1; no longer C10.1
- net GND: now also C1.2, C10.2, C2.2, C23.-, C7.2, C8.2, JP2.1, LED1.C, R1.1, R12.2, R9.1, X1.19; no longer C16.2, C17.2, C19.-, C20.2, C6.2, JP1.1, LED3.C, R14.2, R19.1, R8.1, X2.19
- net ISOGND: now also C15.1, C16.2, C17.-, C19.2, C20.2, LED3.C, R15.2, R9.2, X2.4; no longer C1.2, C2.2, C7.2, C8.-, C9.1, LED1.C, R5.2, R8.2, X1.4
- net ISOVCC: now also C16.1, C17.+, R13.2, R14.1, R8.2; no longer C7.1, C8.+, R1.2, R6.1, R7.2
- net LCD_CK: now also X1.14; no longer X2.14
- net LCD_SI: now also X1.12; no longer X2.12
- net N$10: now also R10.1; no longer R12.1
- net N$15: now also R13.1, R15.1; no longer R1.1, R5.1
- net N$16: now also C4.1; no longer C5.1
- net N$2: now also R1.2, R2.1, R3.1, SW1.2; no longer JP2.2, R18.1, R19.2
- net N$4: now also LED2.A, R11.2; no longer LED3.A, R13.2
- net N$5: now also LED1.A, R10.2; no longer LED2.A, R12.2
- net N$54: now also C20.1, R17.1; no longer C2.1, R3.1
- net N$55: now also C19.1, R16.1; no longer C1.1, R2.1
- net N$6: now also LED3.A, R14.2; no longer LED1.A, R6.2
- net N$9: now also R21.1; no longer R15.1
- net OSC_IN: now also C8.1, Q2.1, R5.1; no longer C11.1, Q1.1, R10.1
- net OSC_IN1: now also C5.1, Q1.4, R4.2; no longer C22.1, Q2.4, R20.2
- net OSC_OUT: now also C10.1, Q2.2, R5.2; no longer C12.1, Q1.2, R10.2
- net OSC_OUT1: now also C2.1, Q1.1, R4.1; no longer C21.1, Q2.1, R20.1
- net PA0: now also X1.3; no longer X2.3
- net PA1: now also X1.4; no longer X2.4
- net PA15: now also X1.20; no longer X2.20
- net PA2: now also X1.5; no longer X2.5
- net PA3: now also X1.6; no longer X2.6
- net PA4: now also X1.7; no longer X2.7
- net PA5: now also X1.8; no longer X2.8
- net PA6: now also X1.9; no longer X2.9
- net PA7: now also X1.10; no longer X2.10
- net PB0: now also X1.11; no longer X2.11
- net PB13: now also X1.15; no longer X2.15
- net PB14: now also X1.16; no longer X2.16
- net PB15: now also X1.17; no longer X2.17
- net PB3: now also X1.18; no longer X2.18
- net SCL1: now also R18.1; no longer R16.1
- net SDA1: now also R19.1; no longer R17.1
- net VBAT: now also JP2.2, X1.2; no longer JP1.2, X2.2
- net VDDA: now also C12.1, R6.2; no longer C13.1, R11.2
Routing:
- net PC13: track 0.00 -> 18.7 mm, vias 0 -> 2
- net +3V3: track 121.0 -> 127.9 mm
- net N$2: track 4.20 -> 7.10 mm
- net BOOT0: track 15.5 -> 14.0 mm
- net !RESET: track 46.1 -> 47.5 mm
- net VBAT: track 16.1 -> 17.4 mm
- net CAN_TX: track 46.8 -> 47.7 mm
- net CAN_RX: track 39.3 -> 40.1 mm
- net GND: vias 54 -> 56
Other:
- board text added: "Rev.B (09/14)"
- board text removed: "Rev.B (07/14)"

Commit message: Add alternative DC-DC B0505S-1W (MornSun, etc)
Parts:
- added DA2': B0505S, dcdc-isolated:SIP4
- moved DA1' 1.27 mm to (54.0, 25.4)
Connections:
- net +5V: now also DA2'.2
- net GND: now also DA2'.1
- net ISOGND: now also DA2'.3
- net ISOVCC: now also DA2'.4
Routing:
- net CAN_TX: track 47.7 -> 49.1 mm
- net CANL: track 24.2 -> 25.5 mm
- net +5V: track 93.5 -> 94.8 mm
- net ISOVCC: track 42.5 -> 43.7 mm
- net CAN_RX: track 40.1 -> 41.3 mm
